File: TPS5430_Experiment.kicad_pcb (KiCad board)
At the start: 2 copper layers, 50 x 50 mm, 21 parts, among them J1 HT5.08, J2 HT5.08, J3 Barrel_Jack, U1 TPS5430DDA

Commit message: 更新原理图
Parts:
- removed TP4: TestPoint, TestPoint:TestPoint_2Pads_Pitch2.54mm_Drill0.8mm
- added C4: 0.1uF, Capacitor_SMD:C_0805_2012Metric_Pad1.18x1.45mm_HandSolder, F.Cu at (132.1, 103.8)
- added C5: 10uF, Capacitor_SMD:C_1206_3216Metric_Pad1.33x1.80mm_HandSolder, F.Cu at (155.8, 90.0)
- added C6: 0.1uF, Capacitor_SMD:C_0805_2012Metric_Pad1.18x1.45mm_HandSolder, F.Cu at (153.3, 90.3)
- added kibuzzard-62F31943: G***, kibuzzard-62F31943, F.Cu at (150.6, 123.5)
- R1: value 3.24kOhm -> 10kOhm
- RV1: value 10kOhm -> 100kOhm
- moved TP1 3.01 mm to (127.0, 87.2)
- moved TP3 2.63 mm to (163.1, 96.8)
- moved TP2 2.53 mm to (135.6, 112.5), turned to -90 degrees
Connections:
- TP1 pad 2: Net-(C2-Pad1) -> GNDREF
- TP2 pad 2: Net-(C1-Pad2) -> GNDREF
- TP3 pad 2: Net-(C3-Pad1) -> GNDREF
Routing:
- net Net-(C3-Pad1): track 9.24 -> 27.4 mm
Other:
- board text added: "Vout"
- board text removed: "5V"
- board text removed: "TPS5430_EXP_V1.3 2022-08-01 by Sage Xiong"
